Commit message: feat: completed agv .urdf as part of agv_description ROS package

File: src/agv_description/urdf/agv.urdf.xacro (robot description, xacro)
@@ -1,4 +1,6 @@
 <?xml version="1.0"?>
-<robot name="agv_3Dlidar" xmlns:xacro="http://www.ros.org/wiki/xacro">
+<robot name="agv" xmlns:xacro="http://www.ros.org/wiki/xacro">
+    <xacro:include filename="$(find agv_description)/urdf/materials.xacro" />
+    <xacro:include filename="$(find agv_description)/urdf/agv.gazebo" />
     <!-- Constants for robot dimensions -->
     <xacro:property name="PI" value="3.1415926535897931"/>
@@ -14,5 +16,5 @@
     <xacro:property name="wheel_rad" value="0.15" /> <!-- radius=0.15 meters-->
     <xacro:property name="wheel_len" value="0.30" /> <!-- length=0.30 meters-->
-    <xacro:macro name="visual_collision_template" params="x y z *shape">
+    <xacro:macro name="visual_collision_template" params="x y z material *shape">
         <visual>
         <origin xyz="${x} ${y} ${z}" rpy="0 0 0"/>
@@ -20,4 +22,5 @@
             <xacro:insert_block name="shape" />
         </geometry>
+        <material name="${material}"/>
         </visual>
         <collision>
@@ -29,11 +32,12 @@
     </xacro:macro>
     <xacro:macro name="wheel_template" params="name x y rad len">
-        <joint name="chassis_${name}_joint" type="fixed">
+        <joint name="chassis_${name}_joint" type="continuous">
             <parent link="chassis"/>
             <child link="${name}"/>
             <origin xyz="${x} ${y} 0.0" rpy="${PI/2} 0 0"/>
+            <axis xyz="0 0 1"/>
         </joint>
         <link name="${name}">
-            <xacro:visual_collision_template x="0.0" y="0.0" z="0.0">
+            <xacro:visual_collision_template x="0.0" y="0.0" z="0.0" material="black">
                 <cylinder radius="${rad}" length="${len}" />
             </xacro:visual_collision_template>
@@ -48,13 +52,7 @@
     </xacro:macro>
     <!-- AGV Description Starts -->
-    <link name="world"/>
-    <joint name="base_world_joint" type="fixed">
-        <parent link="world"/>
-        <child link="base_CoordSys"/>
-        <origin xyz="0.0 0.0 0.0" rpy="0 0 0"/>
-    </joint>
-    <link name="base_CoordSys"/>
+    <link name="agv_CoordSys"/>
     <joint name="base_chassis_joint" type="fixed">
-        <parent link="base_CoordSys"/>
+        <parent link="agv_CoordSys"/>
         <child link="chassis"/>
         <origin xyz="0.0 0.0 ${wheel_rad}" rpy="0 0 0"/>
@@ -63,16 +61,16 @@
     <link name="chassis">
         <!-- Box representing AGV body which contains battery, electronics, etc. -->
-        <xacro:visual_collision_template x="0.0" y="0.0" z="${mast_z/2}">
+        <xacro:visual_collision_template x="0.0" y="0.0" z="${mast_z/2}" material="grey">
             <box size="${mast_x} ${chassis_y} ${mast_z}"/>
         </xacro:visual_collision_template>
         <!-- Box representing AGV mast -->
-        <xacro:visual_collision_template x="${(mast_x+chassis_x)/2}" y="0.0" z="${chassis_z/2}">
+        <xacro:visual_collision_template x="${(mast_x+chassis_x)/2}" y="0.0" z="${chassis_z/2}" material="orange">
             <box size="${chassis_x} ${chassis_y} ${chassis_z}"/>
         </xacro:visual_collision_template>
         <!-- Box representing AGV forks -->
-        <xacro:visual_collision_template x="${-(mast_x+fork_x)/2}" y="${fork_y_offset+fork_y/2}" z="${fork_z/2}">
+        <xacro:visual_collision_template x="${-(mast_x+fork_x)/2}" y="${fork_y_offset+fork_y/2}" z="${fork_z/2}" material="black">
             <box size="${fork_x} ${fork_y} ${fork_z}"/>
         </xacro:visual_collision_template>
-        <xacro:visual_collision_template x="${-(mast_x+fork_x)/2}" y="${-(fork_y_offset+fork_y/2)}" z="${fork_z/2}">
+        <xacro:visual_collision_template x="${-(mast_x+fork_x)/2}" y="${-(fork_y_offset+fork_y/2)}" z="${fork_z/2}" material="black">
             <box size="${fork_x} ${fork_y} ${fork_z}"/>
         </xacro:visual_collision_template>
@@ -89,13 +87,24 @@
     <xacro:wheel_template name="wheelR" x="0" y="${-(chassis_y-wheel_len)/2}" rad="${wheel_rad}" len="${wheel_len}"/>
     <xacro:wheel_template name="wheelC" x="${chassis_x}" y="0" rad="${wheel_rad}" len="${wheel_len}"/>
-    <!-- AGV Lidar Sensor -->
-    <joint name="chassis_lidar_joint" type="fixed">
+    <!-- AGV Lidar3D Sensor -->
+    <joint name="chassis_lidar3D_joint" type="fixed">
         <parent link="chassis"/>
-        <child link="lidar"/>
-        <origin xyz="0.0 0.0 ${mast_z+.15}" rpy="0 0 0"/>
+        <child link="lidar3D"/>
+        <origin xyz="0.0 0.0 ${mast_z+.1}" rpy="0 0 0"/>
     </joint>
-    <link name="lidar">
-        <xacro:visual_collision_template x="0.0" y="0.0" z="0.0">
-            <cylinder radius="0.1" length="0.3" />
+    <link name="lidar3D">
+        <xacro:visual_collision_template x="0.0" y="0.0" z="0.0" material="green">
+            <cylinder radius="0.1" length="0.2" />
+        </xacro:visual_collision_template>
+    </link>
+    <!-- AGV Lidar2D Sensor -->
+    <joint name="chassis_lidar2D_joint" type="fixed">
+        <parent link="chassis"/>
+        <child link="lidar2D"/>
+        <origin xyz="0.0 0.0 ${mast_z+.3}" rpy="0 0 0"/>
+    </joint>
+    <link name="lidar2D">
+        <xacro:visual_collision_template x="0.0" y="0.0" z="0.0" material="red">
+            <cylinder radius="0.1" length="0.2" />
         </xacro:visual_collision_template>
     </link>

Commit message: feat: added differential drive gazebo plugin to the AGV

File: src/agv_description/urdf/agv.urdf.xacro (robot description, xacro)
@@ -1,6 +1,4 @@
 <?xml version="1.0"?>
 <robot name="agv" xmlns:xacro="http://www.ros.org/wiki/xacro">
-    <xacro:include filename="$(find agv_description)/urdf/materials.xacro" />
-    <xacro:include filename="$(find agv_description)/urdf/agv.gazebo.xarco" />
     <!-- Constants for robot dimensions -->
     <xacro:property name="PI" value="3.1415926535897931"/>
@@ -16,4 +14,8 @@
     <xacro:property name="wheel_rad" value="0.15" /> <!-- radius=0.15 meters-->
     <xacro:property name="wheel_len" value="0.30" /> <!-- length=0.30 meters-->
+    <!-- Include other xacro files-->
+    <xacro:include filename="$(find agv_description)/urdf/materials.xacro" />
+    <xacro:include filename="$(find agv_description)/urdf/agv.gazebo.xarco" />
+    <!-- Setup some useful xacro macros-->
     <xacro:macro name="visual_collision_template" params="x y z material *shape">
         <visual>
@@ -35,5 +37,5 @@
             <parent link="chassis"/>
             <child link="${name}"/>
-            <origin xyz="${x} ${y} 0.0" rpy="${PI/2} 0 0"/>
+            <origin xyz="${x} ${y} 0.0" rpy="${-PI/2} 0 0"/>
             <axis xyz="0 0 1"/>
         </joint>

Commit message: feat: simulation pipeline completed. agv_bringup package added to launch complete pipeline

File: src/agv_description/urdf/agv.urdf.xacro (robot description, xacro)
@@ -8,5 +8,5 @@
     <xacro:property name="mast_x" value="0.3" /> <!-- length=0.3 meters -->
     <xacro:property name="mast_z" value="3.0" /> <!-- height=3.0 meters-->
-    <xacro:property name="fork_x" value="2.5" /> <!-- length=2.5 meters-->
+    <xacro:property name="fork_x" value="1.5" /> <!-- length=1.5 meters-->
     <xacro:property name="fork_y" value="0.2" /> <!-- width=0.2 meters-->
     <xacro:property name="fork_z" value="0.05" /> <!-- height=0.05 meters-->
