Commit message: feat: demos for AMR localization while doing navigation.
Localization is done using AMCL. Automatic navigation is done using the
move_base package. A demo with manual navigation using keyboard telop
is also added.

File: robot/agv.urdf.xacro (robot description, xacro)
@@ -14,4 +14,6 @@
     <xacro:property name="wheel_rad" value="0.15" /> <!-- radius=0.15 meters-->
     <xacro:property name="wheel_len" value="0.30" /> <!-- length=0.30 meters-->
+    <xacro:property name="chassis_mass" value="100" /> <!-- mass=100 kg-->
+    <xacro:property name="wheel_mass" value="1" /> <!-- mass=1 kg-->
     <!-- Include other xacro files-->
     <xacro:include filename="$(find factorybot)/robot/materials.xacro" />
@@ -33,5 +35,5 @@
         </collision>
     </xacro:macro>
-    <xacro:macro name="wheel_template" params="name x y rad len">
+    <xacro:macro name="wheel_template" params="name x y rad length mass">
         <joint name="chassis_${name}_joint" type="continuous">
             <parent link="chassis"/>
@@ -42,12 +44,13 @@
         <link name="${name}">
             <xacro:visual_collision_template x="0.0" y="0.0" z="0.0" material="black">
-                <cylinder radius="${rad}" length="${len}" />
+                <cylinder radius="${rad}" length="${length}" />
             </xacro:visual_collision_template>
             <inertial>
             <origin xyz="0 0 0" rpy="0 0 0"/>
-            <mass value="1"/>
-            <inertia ixx="0.0145833" ixy="0" ixz="0"
-                    iyy="0.0145833" iyz="0"
-                    izz="0.0125" />
+            <mass value="${mass}"/>
+            <!-- Cylinder: Izz=(1/2)*m*r^2, Ixx=Iyy=(1/12)*m*(3*r^2+h^2)-->
+            <inertia ixx="${(1/12)*mass*(3*pow(rad,2)+pow(length,2))}" ixy="0" ixz="0"
+                    iyy="${(1/12)*mass*(3*pow(rad,2)+pow(length,2))}" iyz="0"
+                    izz="${.5*mass*pow(rad,2)}" />
             </inertial>
         </link>
@@ -79,5 +82,5 @@
         <inertial>
         <origin xyz="0 0 0" rpy="0 0 0"/>
-        <mass value="100"/>
+        <mass value="${chassis_mass}"/>
         <inertia ixx="60" ixy="0" ixz="0"
                 iyy="60" iyz="0"
@@ -86,7 +89,7 @@
     </link>
     <!-- AGV Wheels -->
-    <xacro:wheel_template name="wheelL" x="0" y="${(chassis_y-wheel_len)/2+.01}" rad="${wheel_rad}" len="${wheel_len}"/>
-    <xacro:wheel_template name="wheelR" x="0" y="${-(chassis_y-wheel_len)/2-.01}" rad="${wheel_rad}" len="${wheel_len}"/>
-    <xacro:wheel_template name="wheelC" x="${chassis_x}" y="0" rad="${wheel_rad}" len="${wheel_len}"/>
+    <xacro:wheel_template name="wheelL" x="0" y="${(chassis_y-wheel_len)/2+.01}" rad="${wheel_rad}" length="${wheel_len}" mass="${wheel_mass}"/>
+    <xacro:wheel_template name="wheelR" x="0" y="${-(chassis_y-wheel_len)/2-.01}" rad="${wheel_rad}" length="${wheel_len}" mass="${wheel_mass}"/>
+    <xacro:wheel_template name="wheelC" x="${chassis_x}" y="0" rad="${wheel_rad}" length="${wheel_len}" mass="${wheel_mass}"/>
     <!-- AGV Lidar3D Sensor -->
     <joint name="chassis_lidar3D_joint" type="fixed">

File: robot/amr.urdf.xacro (robot description, xacro)
@@ -7,6 +7,8 @@
     <xacro:property name="chassis_z" value="0.4" /> <!-- height=0.4 meters-->
     <xacro:property name="caster_rad" value="0.02" />
+    <xacro:property name="chassis_mass" value="100" />
     <xacro:property name="wheel_rad" value="0.15" />
     <xacro:property name="wheel_len" value="0.05" />
+    <xacro:property name="wheel_mass" value="2" />
     <xacro:property name="lidar_rad" value="0.05" />
     <xacro:property name="lidar_len" value="0.08" />
@@ -33,5 +35,5 @@
         </collision>
     </xacro:macro>
-    <xacro:macro name="wheel_template" params="name x y rad len">
+    <xacro:macro name="wheel_template" params="name x y rad length mass">
         <joint name="chassis_${name}_joint" type="continuous">
             <parent link="chassis"/>
@@ -42,12 +44,13 @@
         <link name="${name}">
             <xacro:visual_collision_template x="0.0" y="0.0" z="0.0" material="black">
-                <cylinder radius="${rad}" length="${len}" />
+                <cylinder radius="${rad}" length="${length}" />
             </xacro:visual_collision_template>
             <inertial>
             <origin xyz="0 0 0" rpy="0 0 0"/>
-            <mass value="1"/>
-            <inertia ixx="0.0145833" ixy="0" ixz="0"
-                    iyy="0.0145833" iyz="0"
-                    izz="0.0125" />
+            <mass value="${mass}"/>
+            <!-- Cylinder: Izz=(1/2)*m*r^2, Ixx=Iyy=(1/12)*m*(3*r^2+h^2)-->
+            <inertia ixx="${(1/12)*mass*(3*pow(rad,2)+pow(length,2))}" ixy="0" ixz="0"
+                    iyy="${(1/12)*mass*(3*pow(rad,2)+pow(length,2))}" iyz="0"
+                    izz="${.5*mass*pow(rad,2)}" />
             </inertial>
         </link>
@@ -115,18 +118,19 @@
         <inertial>
         <origin xyz="0 0 0" rpy="0 0 0"/>
-        <mass value="100"/>
-        <inertia ixx="60" ixy="0" ixz="0"
-                iyy="60" iyz="0"
-                izz="60" />
+        <mass value="${chassis_mass}"/>
+        <!-- Box: Ixx=(1/12)*m*(y^2+z^2), Iyy=(1/12)*m*(x^2+z^2), Izz=(1/12)*m*(x^2+y^2)-->
+        <inertia ixx="${(1/12)*chassis_mass*(pow(chassis_y,2)+pow(chassis_z,2))}" ixy="0" ixz="0"
+                iyy="${(1/12)*chassis_mass*(pow(chassis_x,2)+pow(chassis_z,2))}" iyz="0"
+                izz="${(1/12)*chassis_mass*(pow(chassis_x,2)+pow(chassis_y,2))}" />
         </inertial>
     </link>
     <!-- AMR Wheels -->
-    <xacro:wheel_template name="wheelL" x="0" y="${(chassis_y-wheel_len*3.5)/2}" rad="${wheel_rad}" len="${wheel_len}"/>
-    <xacro:wheel_template name="wheelR" x="0" y="${-(chassis_y-wheel_len*3.5)/2}" rad="${wheel_rad}" len="${wheel_len}"/>
+    <xacro:wheel_template name="wheelL" x="0" y="${(chassis_y-wheel_len*3.5)/2}" rad="${wheel_rad}" length="${wheel_len}"  mass="${wheel_mass}"/>
+    <xacro:wheel_template name="wheelR" x="0" y="${-(chassis_y-wheel_len*3.5)/2}" rad="${wheel_rad}" length="${wheel_len}"  mass="${wheel_mass}"/>
     <!-- AMR Lidar2D Sensor (Top Right) -->
     <joint name="chassis_lidar2D_top_right_joint" type="fixed">
         <parent link="chassis"/>
         <child link="lidar2D_TR"/>
-        <origin xyz="${chassis_x/2-lidar_rad} ${chassis_y/2-lidar_rad} ${chassis_z/20+lidar_len/2}" rpy="0 0 0"/>
+        <origin xyz="${chassis_x/2} ${chassis_y/2} ${chassis_z/20+lidar_len/2}" rpy="0 0 0"/>
     </joint>
     <link name="lidar2D_TR">
